File: Circuit imprimé/Axe_linéaire/Connector.kicad_sch (KiCad schematic)
At the start: 5 parts, among them J1 Conn_01x14_Shielded, J2 Conn_01x14_Shielded

Commit message: circuit V1
Parts:
- D3: renamed from D?; footprint (none) -> LED_SMD:LED_1206_3216Metric
- J3: renamed from J?; footprint (none) -> Connector_Card:microSD_HC_Hirose_DM3AT-SF-PEJM5
- R9: renamed from R?; footprint (none) -> Resistor_SMD:R_0805_2012Metric
Connections:
- net VDC is gone; now on net +3V3: J2.13 (Pin_13), J2.14 (Pin_14)
- net GND: now also J3.11 (SHIELD)
Changed lines of the file:
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@@
     (stroke (width 0) (type default) (color 0 0 0 0))
   )
-  (wire (pts (xy 115.57 17.78) (xy 115.57 20.32))
+  (wire (pts (xy 116.84 16.51) (xy 115.57 20.32))
     (stroke (width 0) (type default) (color 0 0 0 0))
   )
@@
   )
   (wire (pts (xy 115.57 50.8) (xy 115.57 53.34))
+    (stroke (width 0) (type default) (color 0 0 0 0))
+  )
+  (wire (pts (xy 283.21 46.99) (xy 283.21 48.26))
     (stroke (width 0) (type default) (color 0 0 0 0))
   )
@@
     (pin "1")
   )
-  (symbol (lib_id "power:VDC") (at 115.57 17.78 0) (unit 1)
-    (in_bom yes) (on_board yes) (fields_autoplaced)
-    (property "Reference" "#PWR042" (id 0) (at 115.57 20.32 0)
-      (effects (font (size 1.27 1.27)) hide)
-    )
-    (property "Value" "VDC" (id 1) (at 115.57 12.7 0))
-    (property "Footprint" "" (id 2) (at 115.57 17.78 0)
-      (effects (font (size 1.27 1.27)) hide)
-    )
-    (property "Datasheet" "" (id 3) (at 115.57 17.78 0)
+  (symbol (lib_id "power:GND") (at 283.21 48.26 0) (unit 1)
+    (in_bom yes) (on_board yes) (fields_autoplaced)
+    (property "Reference" "#PWR0104" (id 0) (at 283.21 54.61 0)
+      (effects (font (size 1.27 1.27)) hide)
+    )
+    (property "Value" "GND" (id 1) (at 283.21 53.34 0))
+    (property "Footprint" "" (id 2) (at 283.21 48.26 0)
+      (effects (font (size 1.27 1.27)) hide)
+    )
+    (property "Datasheet" "" (id 3) (at 283.21 48.26 0)
       (effects (font (size 1.27 1.27)) hide)
     )
@@
   (symbol (lib_id "Connector:Micro_SD_Card_Det") (at 262.89 34.29 0) (unit 1)
     (in_bom yes) (on_board yes) (fields_autoplaced)
-    (property "Reference" "J?" (id 0) (at 263.525 12.7 0))
+    (property "Reference" "J3" (id 0) (at 263.525 12.7 0))
     (property "Value" "Micro_SD_Card_Det" (id 1) (at 263.525 15.24 0))
-    (property "Footprint" "" (id 2) (at 314.96 16.51 0)
+    (property "Footprint" "Connector_Card:microSD_HC_Hirose_DM3AT-SF-PEJM5" (id 2) (at 314.96 16.51 0)
       (effects (font (size 1.27 1.27)) hide)
     )
@@
   (symbol (lib_id "Device:R") (at 214.63 44.45 90) (unit 1)
     (in_bom yes) (on_board yes)
-    (property "Reference" "R?" (id 0) (at 214.63 38.1 90))
+    (property "Reference" "R9" (id 0) (at 214.63 38.1 90))
     (property "Value" "30" (id 1) (at 214.63 44.45 90))
-    (property "Footprint" "" (id 2) (at 214.63 46.228 90)
+    (property "Footprint" "Resistor_SMD:R_0805_2012Metric" (id 2) (at 214.63 46.228 90)
       (effects (font (size 1.27 1.27)) hide)
     )
@@
   (symbol (lib_id "Device:LED") (at 209.55 36.83 90) (unit 1)
     (in_bom yes) (on_board yes)
-    (property "Reference" "D?" (id 0) (at 213.36 37.1474 90)
+    (property "Reference" "D3" (id 0) (at 213.36 37.1474 90)
       (effects (font (size 1.27 1.27)) (justify right))
     )
@@
       (effects (font (size 1.27 1.27)) (justify right))
     )
-    (property "Footprint" "" (id 2) (at 209.55 36.83 0)
+    (property "Footprint" "LED_SMD:LED_1206_3216Metric" (id 2) (at 209.55 36.83 0)
       (effects (font (size 1.27 1.27)) hide)
     )
@@
   (symbol (lib_id "power:+3V3") (at 209.55 33.02 0) (unit 1)
     (in_bom yes) (on_board yes) (fields_autoplaced)
-    (property "Reference" "#PWR?" (id 0) (at 209.55 36.83 0)
+    (property "Reference" "#PWR0101" (id 0) (at 209.55 36.83 0)
       (effects (font (size 1.27 1.27)) hide)
     )
@@
     )
     (property "Datasheet" "" (id 3) (at 209.55 33.02 0)
+      (effects (font (size 1.27 1.27)) hide)
+    )
+    (pin "1")
+  )
+  (symbol (lib_id "power:+3V3") (at 116.84 16.51 0) (unit 1)
+    (in_bom yes) (on_board yes) (fields_autoplaced)
+    (property "Reference" "#PWR0113" (id 0) (at 116.84 20.32 0)
+      (effects (font (size 1.27 1.27)) hide)
+    )
+    (property "Value" "+3V3" (id 1) (at 116.84 11.43 0))
+    (property "Footprint" "" (id 2) (at 116.84 16.51 0)
+      (effects (font (size 1.27 1.27)) hide)
+    )
+    (property "Datasheet" "" (id 3) (at 116.84 16.51 0)
       (effects (font (size 1.27 1.27)) hide)
     )
@@
   (symbol (lib_id "power:+3.3V") (at 227.33 31.75 0) (unit 1)
     (in_bom yes) (on_board yes)
-    (property "Reference" "#PWR?" (id 0) (at 227.33 35.56 0)
+    (property "Reference" "#PWR0105" (id 0) (at 227.33 35.56 0)
       (effects (font (size 1.27 1.27)) hide)
     )
@@
   (symbol (lib_id "power:GND") (at 240.03 48.26 0) (unit 1)
     (in_bom yes) (on_board yes) (fields_autoplaced)
-    (property "Reference" "#PWR?" (id 0) (at 240.03 54.61 0)
+    (property "Reference" "#PWR0102" (id 0) (at 240.03 54.61 0)
       (effects (font (size 1.27 1.27)) hide)
     )
@@
   (symbol (lib_id "power:GND") (at 223.52 39.37 0) (unit 1)
     (in_bom yes) (on_board yes) (fields_autoplaced)
-    (property "Reference" "#PWR?" (id 0) (at 223.52 45.72 0)
-      (effects (font (size 1.27 1.27)) hide)
-    )
+    (property "Reference" "#PWR0103" (id 0) (at 223.52 45.72 0)
+      (effects (font (size 1.27 1.27)) hide)
+    )

Commit message: tout mes CI sont pret
Connections:
- net +3V3 is gone; now on net +3.3V: D3.2 (A), J2.13 (Pin_13), J2.14 (Pin_14)
- net INT2_Haut: now reaches J2.8 (Pin_8)
- net INT1_Haut: now reaches J2.9 (Pin_9)
Changed lines of the file:
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@@
+    )
+  )
+  (global_label "INT1_Haut" (shape output) (at 115.57 33.02 0) (fields_autoplaced)
+    (effects (font (size 1.27 1.27)) (justify left))
+    (property "Intersheet References" "${INTERSHEET_REFS}" (id 0) (at 127.4174 32.9406 0)
+      (effects (font (size 1.27 1.27)) (justify left) hide)
     )
   )
@@
     (property "Intersheet References" "${INTERSHEET_REFS}" (id 0) (at 230.4202 26.5906 0)
       (effects (font (size 1.27 1.27)) (justify right) hide)
+    )
+  )
+  (global_label "INT2_Haut" (shape output) (at 115.57 35.56 0) (fields_autoplaced)
+    (effects (font (size 1.27 1.27)) (justify left))
+    (property "Intersheet References" "${INTERSHEET_REFS}" (id 0) (at 127.4174 35.4806 0)
+      (effects (font (size 1.27 1.27)) (justify left) hide)
     )
   )
@@
     )
     (property "Datasheet" "" (id 3) (at 17.78 17.78 0)
+      (effects (font (size 1.27 1.27)) hide)
+    )
+    (pin "1")
+  )
+  (symbol (lib_id "power:+3.3V") (at 116.84 16.51 0) (unit 1)
+    (in_bom yes) (on_board yes) (fields_autoplaced)
+    (property "Reference" "#PWR0101" (id 0) (at 116.84 20.32 0)
+      (effects (font (size 1.27 1.27)) hide)
+    )
+    (property "Value" "+3.3V" (id 1) (at 116.84 11.43 0))
+    (property "Footprint" "" (id 2) (at 116.84 16.51 0)
+      (effects (font (size 1.27 1.27)) hide)
+    )
+    (property "Datasheet" "" (id 3) (at 116.84 16.51 0)
       (effects (font (size 1.27 1.27)) hide)
     )
@@
     (pin "9")
   )
+  (symbol (lib_id "power:+3.3V") (at 209.55 33.02 0) (unit 1)
+    (in_bom yes) (on_board yes) (fields_autoplaced)
+    (property "Reference" "#PWR0107" (id 0) (at 209.55 36.83 0)
+      (effects (font (size 1.27 1.27)) hide)
+    )
+    (property "Value" "+3.3V" (id 1) (at 209.55 27.94 0))
+    (property "Footprint" "" (id 2) (at 209.55 33.02 0)
+      (effects (font (size 1.27 1.27)) hide)
+    )
+    (property "Datasheet" "" (id 3) (at 209.55 33.02 0)
+      (effects (font (size 1.27 1.27)) hide)
+    )
+    (pin "1")
+  )
   (symbol (lib_id "power:GND") (at 105.41 15.24 0) (unit 1)
     (in_bom yes) (on_board yes) (fields_autoplaced)
@@
       (effects (font (size 1.27 1.27)) hide)
     )
-    (pin "1")
-  )
-  (symbol (lib_id "power:+3V3") (at 209.55 33.02 0) (unit 1)
-    (in_bom yes) (on_board yes) (fields_autoplaced)
-    (property "Reference" "#PWR0101" (id 0) (at 209.55 36.83 0)
-      (effects (font (size 1.27 1.27)) hide)
-    )
-    (property "Value" "+3V3" (id 1) (at 209.55 27.94 0))
-    (property "Footprint" "" (id 2) (at 209.55 33.02 0)
-      (effects (font (size 1.27 1.27)) hide)
-    )
-    (property "Datasheet" "" (id 3) (at 209.55 33.02 0)
-      (effects (font (size 1.27 1.27)) hide)
-    )
-    (pin "1")
-  )
-  (symbol (lib_id "power:+3V3") (at 116.84 16.51 0) (unit 1)
-    (in_bom yes) (on_board yes) (fields_autoplaced)
-    (property "Reference" "#PWR0113" (id 0) (at 116.84 20.32 0)
-      (effects (font (size 1.27 1.27)) hide)
-    )
-    (property "Value" "+3V3" (id 1) (at 116.84 11.43 0))
-    (property "Footprint" "" (id 2) (at 116.84 16.51 0)
-      (effects (font (size 1.27 1.27)) hide)
-    )
-    (property "Datasheet" "" (id 3) (at 116.84 16.51 0)
-      (effects (font (size 1.27 1.27)) hide)
-    )
