File: Circuit imprimé/Axe_linéaire/Axe_linéaire.kicad_pcb (KiCad board)
At the start: 2 copper layers, 77 x 54 mm, 4 parts

Commit message: circuit V1
Parts:
- removed the REF** at (172.5, 60.5)
- added C1: 100n, Library:Cap 100nf 0805, F.Cu at (114.0, 105.9)
- added C2: 100n, Library:Cap 100nf 0805, F.Cu at (116.5, 105.8)
- added C3: 10u, Capacitor_SMD:CP_Elec_6.3x7.7, F.Cu at (110.0, 68.5)
- added C4: 10u, Capacitor_SMD:CP_Elec_6.3x7.7, F.Cu at (169.0, 61.0)
- added C5: 100n, Library:Cap 100nf 0805, F.Cu at (153.8, 59.0)
- added D1: D_Zener, Library:SOD223, F.Cu at (157.3, 61.0)
- added D2: LED, Library:UV_LED, F.Cu at (140.0, 103.5)
- added D3: LED, LED_SMD:LED_1206_3216Metric, F.Cu at (154.0, 68.5)
- added FB1: FerriteBead, Library:ferrite Bead, F.Cu at (156.5, 59.5)
- added J1: Conn_01x14_Shielded, Library:FPC 2x7 p=1mm, F.Cu at (161.5, 81.9)
- added J2: Conn_01x14_Shielded, Library:FPC 2x7 p=1mm, F.Cu at (162.0, 103.4)
- added J3: Micro_SD_Card_Det, Connector_Card:microSD_HC_Hirose_DM3AT-SF-PEJM5, F.Cu at (144.5, 66.0)
- added JP1: SolderJumper_3_Bridged12, Jumper:SolderJumper-3_P1.3mm_Bridged12_RoundedPad1.0x1.5mm, F.Cu at (119.0, 105.5)
- added JP2: SolderJumper_2_Open, Jumper:SolderJumper-2_P1.3mm_Open_RoundedPad1.0x1.5mm, F.Cu at (108.5, 103.5)
- added Q1: LP2301LT1G, Package_TO_SOT_SMD:SOT-23, F.Cu at (103.0, 71.0)
- added Q2: LP2301LT1G, Package_TO_SOT_SMD:SOT-23, F.Cu at (158.5, 64.0)
- added R1: 10k, Resistor_SMD:R_0603_1608Metric, F.Cu at (109.5, 106.5)
- added R10: 1k, Resistor_SMD:R_0603_1608Metric, F.Cu at (172.5, 98.5)
- added R11: 1k, Resistor_SMD:R_0603_1608Metric, F.Cu at (171.0, 98.5)
- added R12: 30, Resistor_SMD:R_0805_2012Metric, F.Cu at (163.6, 108.2)
- added R2: 1k, Resistor_SMD:R_0603_1608Metric, F.Cu at (159.6, 58.9)
- added R3: 100, Resistor_SMD:R_0603_1608Metric, F.Cu at (167.0, 108.6)
- added R4: 1k, Resistor_SMD:R_0603_1608Metric, F.Cu at (172.5, 101.5)
- added R5: 1k, Resistor_SMD:R_0603_1608Metric, F.Cu at (171.0, 101.5)
- added R6: 4.7k, Resistor_SMD:R_0603_1608Metric, F.Cu at (113.0, 101.0)
- added R7: 4.7k, Resistor_SMD:R_0603_1608Metric, F.Cu at (116.0, 101.0)
- added R8: 100, Resistor_SMD:R_0603_1608Metric, F.Cu at (135.1, 102.5)
- added R9: 30, Resistor_SMD:R_0805_2012Metric, F.Cu at (154.0, 64.0)
- added SW1: RESET, Library:Tactile Button, F.Cu at (129.5, 69.0)
- added TP1: TestPoint, TestPoint:TestPoint_Pad_D2.0mm, F.Cu at (122.8, 105.2)
- added TP2: TestPoint, TestPoint:TestPoint_Pad_D2.0mm, F.Cu at (155.2, 102.5)
- added TP3: TestPoint, TestPoint:TestPoint_Pad_D2.0mm, F.Cu at (158.8, 102.5)
- added TP4: TestPoint, TestPoint:TestPoint_Pad_D2.0mm, F.Cu at (108.2, 100.8)
- added TP5: TestPoint, TestPoint:TestPoint_Pad_D2.0mm, F.Cu at (121.2, 100.8)
- added U1: PicoW, RPi_Pico:RPi_PicoW_SMD_TH, F.Cu at (126.0, 87.5)
- added U2: LSM6DSRTR, Library:LGA-14_2.5X3X0.86_, F.Cu at (114.5, 104.0)
- added U3: Vishay_TCUT1350X01, Library:Vishay TCUT1350X01, F.Cu at (171.3, 106.8)
- added U4: 74LVC3G17, Package_SO:VSSOP-8_2.3x2mm_P0.5mm, F.Cu at (157.0, 106.8)
Routing:
- net UART_TX: track 0.00 -> 72.2 mm, vias 0 -> 2
- net SDA: track 0.00 -> 67.9 mm, vias 0 -> 1
- net UART_RX: track 0.00 -> 66.8 mm, vias 0 -> 2
- net SCL: track 0.00 -> 62.7 mm, vias 0 -> 2
- net VDC: track 0.00 -> 60.9 mm, vias 0 -> 2
- net +3.3V: track 0.00 -> 40.8 mm, vias 0 -> 12
- net Motor_B: track 0.00 -> 39.5 mm, vias 0 -> 2
- net Motor_A: track 0.00 -> 38.9 mm, vias 0 -> 2
- net SD_CD: track 0.00 -> 35.0 mm
- net Motor_EN: track 0.00 -> 32.5 mm, vias 0 -> 4
- net Emitter1: track 0.00 -> 28.2 mm, vias 0 -> 1
- net Net-(R4-Pad1): track 0.00 -> 25.1 mm
- net Net-(U4-Pad1): track 0.00 -> 24.9 mm
- net GND: track 0.00 -> 23.0 mm, vias 0 -> 1
- net SD_CS: track 0.00 -> 22.4 mm
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- added copper zone on B.Cu, net +3.3V
- added copper zone on F.Cu, net GND
Other:
- outline, holes or cut-outs redrawn

Commit message: 1er circuit fini, schéma de la base fini
Parts:
- moved SW1 0.50 mm to (129.5, 68.5)
Routing:
- net +3.3V: track 40.8 -> 35.1 mm, vias 12 -> 15
- net GND: track 23.0 -> 28.6 mm
- net Net-(U4-Pad1): track 24.9 -> 25.1 mm, vias 0 -> 2

Commit message: tout mes CI sont pret
Parts:
- added G***: LOGO, LOGO, F.Cu at (117.0, 67.5)
- added G***: LOGO, LOGO, F.Cu at (117.5, 86.0)
Connections:
- J2 pad 8: unconnected-(J2-Pad8) -> INT2_Haut
- J2 pad 9: unconnected-(J2-Pad9) -> INT1_Haut
- U1 pad 10: unconnected-(U1-Pad10) -> INT2_Haut
- U1 pad 9: unconnected-(U1-Pad9) -> INT1_Haut
Routing:
- net INT1_Haut: track 0.00 -> 52.8 mm, vias 0 -> 2
- net INT2_Haut: track 0.00 -> 42.6 mm, vias 0 -> 2
- net Net-(R4-Pad1): track 25.1 -> 29.5 mm, vias 0 -> 2
Other:
- board text added: "FRAMBOURT Mateïs BOCQUILLON Noé"
- board text added: "TIPE 2023"
- board text added: "https://github.com/Docredstein/TIPE_TMD"
