File: Circuit imprimé/base/base.kicad_pcb (KiCad board)
At the start: 2 copper layers, 70 x 45 mm, 34 parts, among them IC1 L6225DTR, J1 Barrel_Jack_Switch, J2 USB_B, J3 Screw_Terminal_01x02, J4 Conn_01x14_Shielded, J5 UART, Q1 LP2301LT1G, U1 CH340C, U2 AMS1117-3.3

Commit message: tout mes CI sont pret
Parts:
- added G***: LOGO, LOGO, F.Cu at (171.5, 75.0)
Other:
- board text added: "3-12V"
