File: Circuit imprimé/base/base.kicad_sch (KiCad schematic)
At the start: 27 parts, among them IC1 L6225DTR, J1 Barrel_Jack, J2 USB_B, J4 Conn_01x14_Shielded, Q1 LP2301LT1G, U1 CH340C, U2 AMS1117-3.3

Commit message: fin du circuit de base
Parts:
- removed C2: C_Polarized, symbol Device:C_Polarized
- removed J1: Barrel_Jack, symbol Connector:Barrel_Jack
- added D6: LED, LED_SMD:LED_1206_3216Metric, symbol Device:LED
- added J1: Barrel_Jack_Switch, Connector_BarrelJack:BarrelJack_GCT_DCJ200-10-A_Horizontal, symbol Connector:Barrel_Jack_Switch
- added J5: Conn_01x04_Female, Connector_PinSocket_2.54mm:PinSocket_1x04_P2.54mm_Horizontal, symbol Connector:Conn_01x04_Female
- added R8: 1k, Resistor_SMD:R_0603_1608Metric, symbol Device:R
- C1: value C_Polarized -> 10u; footprint (none) -> Capacitor_SMD:CP_Elec_6.3x7.7
- C3, C4: footprint (none) -> Library:Cap 100nf 0805
- C5, C6: footprint (none) -> Capacitor_SMD:C_0805_2012Metric
- C7: footprint (none) -> Capacitor_SMD:C_0603_1608Metric
- D4, D5: footprint (none) -> Diode_SMD:D_SOD-323
- J2: footprint (none) -> Connector_USB:USB_B_OST_USB-B1HSxx_Horizontal
- R1, R2, R6, R7: footprint (none) -> Resistor_SMD:R_0603_1608Metric
- gave numbers to parts that had none: 1
Connections:
- net +VDC: now also J5.4 (Pin_4)
- net GND: now also C1.2, R4.2, R5.1, U2.1 (GND), D6.1 (K), J1.2, J5.3 (Pin_3)
- net UART_RX: now also J5.1 (Pin_1)
- net UART_TX: now also J5.2 (Pin_2)
- net V_Barrel: now also J1.1
- net D-: now reaches J2.2 (D-), U1.6 (UD-)
- net D+: now reaches J2.3 (D+), U1.5 (UD+)
- new net: D6.2 (A), R8.2
- new net Power_led: J1.3, R8.1
- no-connect marks 10 -> 11

Commit message: Passage ENS
Other:
- title: (none) -> Base fixe
