File: Circuit imprimé/assemblage/assemblage.kicad_pcb (KiCad board)
At the start: 2 copper layers, 101 x 101 mm, 108 parts, among them IC1 L6225DTR, J1 Barrel_Jack_Switch, J1 Conn_01x14_Shielded, J2 Conn_01x06_Male, J2 Conn_01x14_Shielded, J2 USB_B, J3 Micro_SD_Card_Det, J3 Screw_Terminal_01x02, J4 Conn_01x14_Shielded, J5 UART, Q1 LP2301LT1G, Q2 LP2301LT1G, SW1 RESET, U1 CH340C, U1 LSM6DSRTR, U1 PicoW, U2 AMS1117-3.3, U2 LSM6DSRTR, U3 Vishay_TCUT1350X01, U4 74LVC3G17

Commit message: circuit imprimé commandé
Parts:
- moved C1 0.71 mm to (217.2, 107.0)
- moved C2 0.71 mm to (217.5, 104.5)
- moved D1 0.71 mm to (221.7, 113.3)
- moved G*** 0.71 mm to (214.0, 114.5)
- moved J1 0.71 mm to (209.7, 115.3)
- moved J2 0.71 mm to (204.0, 111.8)
- moved JP1 0.71 mm to (216.5, 101.0)
- moved JP2 0.71 mm to (214.5, 110.7)
- moved R1 0.71 mm to (217.0, 112.8)
- moved R2 0.71 mm to (219.0, 115.6)
- moved REF** 0.71 mm to (220.5, 121.5)
- moved REF** 0.71 mm to (220.5, 91.5)
- moved REF** 0.71 mm to (207.5, 121.5)
- moved REF** 0.71 mm to (207.5, 91.5)
- moved U1 0.71 mm to (215.5, 106.5)
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Other:
- board size 101 x 101 mm -> 101.5 x 101 mm
